File: CNCPlotter.sch (EAGLE design)
At the start: 126 parts, among them IC1 HEF4050B, IC2 MC34063, IC3 LD111733, IC4 74HC4094, IC5 ATmega32U4, IC6 DRV8811, IC7 DRV8811, J1 Servo, J10 Touchscreen, J11 Touchscreen, J12 X Motor, J13 MS1, J14 MS0, J15 Y Motor, J16 MS1, J17 MS0, J2 Z Drive, J3 ISP, J4 UART, J5 12V Supply, J6 MicroSD Card, J7 HWB, J8 USB, J9 Home Switches, Q1 16MHz

Commit message: Removed CNCPlotter files
Parts:
- J1: value Servo -> SERVO
- J12: value X Motor -> X-MOTOR
- J15: value Y Motor -> Y-MOTOR
- J2: value Z Drive -> Z-DRIVE
- J5: device SparkFun:POWER_JACKSLT -> freetronics-master-v1.1:POWER_JACKPTH
- J8: value USB -> USB-6PSMT; device freetronics-luke:USB-FT -> freetronics-jon:USB-6PSMT
Connections:
- net GND: now also J5.GNDBREAK, J8.FIX1, J8.FIX2, J8.PIN1, J8.PIN2, J8.TAB1, J8.TAB2; no longer J8.SH$1
Changed lines of the file:
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@@
 <?xml version="1.0" encoding="utf-8"?>
 <!DOCTYPE eagle SYSTEM "eagle.dtd">
-<eagle version="6.3">
+<eagle version="6.2">
 <drawing>
 <settings>
@@
 <part name="J7" library="freetronics-luke" deviceset="SJ" device="" value="HWB"/>
 <part name="U$28" library="freetronics-luke" deviceset="GND" device=""/>
-<part name="J8" library="freetronics-luke" deviceset="USB-FT" device="" value="USB"/>
 <part name="Z1" library="freetronics-luke" deviceset="PGB102ST23" device=""/>
 <part name="U$66" library="freetronics-luke" deviceset="GND" device=""/>
@@
 <part name="U$83" library="freetronics-luke" deviceset="GND" device=""/>
 <part name="U$84" library="freetronics-luke" deviceset="GND" device=""/>
-<part name="J1" library="con-molex" deviceset="22-23-2031" device="" value="Servo"/>
+<part name="J1" library="con-molex" deviceset="22-23-2031" device="" value="SERVO"/>
 <part name="J11" library="SparkFun" deviceset="DS_TOUCH_CONNECTOR" device="" value="Touchscreen"/>
 <part name="U$86" library="freetronics-luke" deviceset="GND" device=""/>
@@
 <part name="U$46" library="freetronics-luke" deviceset="+5V" device=""/>
 <part name="P+6" library="supply1" deviceset="+12V" device=""/>
-<part name="J12" library="con-phoenix-254" deviceset="MPT4" device="" value="X Motor">
+<part name="J12" library="con-phoenix-254" deviceset="MPT4" device="" value="X-MOTOR">
 <attribute name="MF" value=""/>
 <attribute name="MPN" value=""/>
@@
 <part name="U$3" library="freetronics-luke" deviceset="+5V" device=""/>
 <part name="P+1" library="supply1" deviceset="+12V" device=""/>
-<part name="J15" library="con-phoenix-254" deviceset="MPT4" device="" value="Y Motor">
+<part name="J15" library="con-phoenix-254" deviceset="MPT4" device="" value="Y-MOTOR">
 <attribute name="MF" value=""/>
 <attribute name="MPN" value=""/>
@@
 <part name="C25" library="rcl" deviceset="CPOL-EU" device="E2.5-6" value="100uF"/>
 <part name="U$106" library="freetronics-luke" deviceset="GND" device=""/>
-<part name="J5" library="SparkFun" deviceset="POWER_JACK" device="SLT" value="12V Supply"/>
+<part name="J5" library="freetronics-master-v1.1" deviceset="POWER_JACK" device="PTH" value="12V Supply"/>
 <part name="C7" library="freetronics-master-v1" deviceset="CAP" device="0603" value="100nF"/>
 <part name="C8" library="freetronics-master-v1" deviceset="CAP" device="0603" value="100nF"/>
@@
 <part name="J4" library="pinhead" deviceset="PINHD-1X4" device="" value="UART"/>
 <part name="J9" library="con-phoenix-254" deviceset="MPT6" device="" value="Home Switches"/>
-<part name="J2" library="con-phoenix-254" deviceset="MPT5" device="" value="Z Drive"/>
+<part name="J2" library="con-phoenix-254" deviceset="MPT5" device="" value="Z-DRIVE"/>
+<part name="J8" library="freetronics-jon" deviceset="USB-6P" device="SMT"/>
 </parts>
 <sheets>
@@
 </instance>
 <instance part="U$28" gate="G$1" x="182.88" y="495.3" rot="MR0"/>
-<instance part="J8" gate="G$1" x="48.26" y="487.68"/>
 <instance part="Z1" gate="G$1" x="63.5" y="480.06" smashed="yes" rot="MR0">
 <attribute name="NAME" x="58.42" y="472.44" size="1.27" layer="95"/>
@@
 <instance part="U$66" gate="G$1" x="55.88" y="469.9" rot="MR0"/>
 <instance part="U$67" gate="G$1" x="63.5" y="469.9" rot="MR0"/>
-<instance part="U$68" gate="G$1" x="43.18" y="469.9" rot="MR0"/>
+<instance part="U$68" gate="G$1" x="43.18" y="467.36" rot="MR0"/>
 <instance part="Q1" gate="G$1" x="96.52" y="469.9" smashed="yes" rot="R90">
 <attribute name="NAME" x="93.98" y="472.44" size="1.27" layer="95"/>
@@
 <attribute name="VALUE" x="231.14" y="721.36" size="1.27" layer="96"/>
 </instance>
+<instance part="J8" gate="G$1" x="45.72" y="487.68" rot="R180"/>
 </instances>
 <busses>
@@
 </segment>
 <segment>
-<pinref part="J8" gate="G$1" pin="SH$1"/>
 <pinref part="U$68" gate="G$1" pin="GND"/>
-<wire x1="43.18" y1="477.52" x2="43.18" y2="472.44" width="0.1524" layer="91"/>
-</segment>
-<segment>
+<wire x1="43.18" y1="474.98" x2="43.18" y2="469.9" width="0.1524" layer="91"/>
+<pinref part="J8" gate="G$1" pin="FIX2"/>
+<pinref part="J8" gate="G$1" pin="TAB2"/>
+<wire x1="45.72" y1="474.98" x2="45.72" y2="469.9" width="0.1524" layer="91"/>
+<wire x1="45.72" y1="469.9" x2="43.18" y2="469.9" width="0.1524" layer="91"/>
+<pinref part="J8" gate="G$1" pin="PIN2"/>
+<wire x1="50.8" y1="480.06" x2="50.8" y2="469.9" width="0.1524" layer="91"/>
+<wire x1="50.8" y1="469.9" x2="45.72" y2="469.9" width="0.1524" layer="91"/>
+<pinref part="J8" gate="G$1" pin="PIN1"/>
+<wire x1="50.8" y1="495.3" x2="50.8" y2="505.46" width="0.1524" layer="91"/>
+<wire x1="50.8" y1="505.46" x2="45.72" y2="505.46" width="0.1524" layer="91"/>
+<wire x1="45.72" y1="505.46" x2="43.18" y2="505.46" width="0.1524" layer="91"/>
+<wire x1="43.18" y1="505.46" x2="35.56" y2="505.46" width="0.1524" layer="91"/>
+<wire x1="35.56" y1="505.46" x2="35.56" y2="469.9" width="0.1524" layer="91"/>
+<wire x1="35.56" y1="469.9" x2="43.18" y2="469.9" width="0.1524" layer="91"/>
+<pinref part="J8" gate="G$1" pin="TAB1"/>
+<wire x1="45.72" y1="500.38" x2="45.72" y2="505.46" width="0.1524" layer="91"/>
+<pinref part="J8" gate="G$1" pin="FIX1"/>
+<wire x1="43.18" y1="500.38" x2="43.18" y2="505.46" width="0.1524" layer="91"/>
+<junction x="43.18" y="505.46"/>
+<junction x="45.72" y="505.46"/>
+<junction x="43.18" y="469.9"/>
+<junction x="45.72" y="469.9"/>
+</segment>
+<segment>
+<pinref part="U$66" gate="G$1" pin="GND"/>
+<wire x1="50.8" y1="482.6" x2="55.88" y2="482.6" width="0.1524" layer="91"/>
+<wire x1="55.88" y1="482.6" x2="55.88" y2="472.44" width="0.1524" layer="91"/>
 <pinref part="J8" gate="G$1" pin="GND"/>
-<pinref part="U$66" gate="G$1" pin="GND"/>
-<wire x1="53.34" y1="482.6" x2="55.88" y2="482.6" width="0.1524" layer="91"/>
-<wire x1="55.88" y1="482.6" x2="55.88" y2="472.44" width="0.1524" layer="91"/>
 </segment>
 <segment>
@@
 <wire x1="27.94" y1="662.94" x2="27.94" y2="647.7" width="0.1524" layer="91"/>
 <wire x1="25.4" y1="662.94" x2="27.94" y2="662.94" width="0.1524" layer="91"/>
+<pinref part="J5" gate="G$1" pin="GNDBREAK"/>
+<wire x1="25.4" y1="665.48" x2="27.94" y2="665.48" width="0.1524" layer="91"/>
+<wire x1="27.94" y1="665.48" x2="27.94" y2="662.94" width="0.1524" layer="91"/>
+<junction x="27.94" y="662.94"/>
 </segment>
 <segment>
@@
 <net name="N$33" class="0">
 <segment>
-<pinref part="J8" gate="G$1" pin="D+"/>
-<wire x1="53.34" y1="487.68" x2="66.04" y2="487.68" width="0.1524" layer="91"/>
+<wire x1="50.8" y1="487.68" x2="66.04" y2="487.68" width="0.1524" layer="91"/>
 <pinref part="Z1" gate="G$1" pin="P$1"/>
 <wire x1="66.04" y1="485.14" x2="66.04" y2="487.68" width="0.1524" layer="91"/>
@@
 <wire x1="68.58" y1="487.68" x2="66.04" y2="487.68" width="0.1524" layer="91"/>
 <pinref part="R16" gate="G$1" pin="2"/>
+<pinref part="J8" gate="G$1" pin="D+"/>
 </segment>
 </net>
 <net name="N$34" class="0">
 <segment>
-<pinref part="J8" gate="G$1" pin="D-"/>
-<wire x1="53.34" y1="490.22" x2="60.96" y2="490.22" width="0.1524" layer="91"/>
+<wire x1="50.8" y1="490.22" x2="60.96" y2="490.22" width="0.1524" layer="91"/>
 <pinref part="Z1" gate="G$1" pin="P$2"/>
 <wire x1="60.96" y1="490.22" x2="63.5" y2="492.76" width="0.1524" layer="91"/>
@@
 <junction x="60.96" y="490.22"/>
 <pinref part="R15" gate="G$1" pin="2"/>
+<pinref part="J8" gate="G$1" pin="D-"/>
 </segment>
 </net>
@@
 <net name="N$2" class="0">
 <segment>
-<pinref part="J8" gate="G$1" pin="VBUS"/>
-<wire x1="53.34" y1="492.76" x2="58.42" y2="492.76" width="0.1524" layer="91"/>
+<wire x1="50.8" y1="492.76" x2="58.42" y2="492.76" width="0.1524" layer="91"/>
 <pinref part="F1" gate="G$1" pin="P$1"/>
 <wire x1="58.42" y1="492.76" x2="58.42" y2="513.08" width="0.1524" layer="91"/>
 <wire x1="58.42" y1="513.08" x2="60.96" y2="513.08" width="0.1524" layer="91"/>
-</segment>
-</net>
+<pinref part="J8" gate="G$1" pin="VBUS"/>
+</segment>
+</net>
