File: STEPDUINO.sch (EAGLE design)
At the start: 126 parts, among them IC1 HEF4050B, IC2 MC34063, IC3 LD111733, IC4 74HC4094, IC5 ATmega32U4, IC6 DRV8811, IC7 DRV8811, J1 SERVO, J10 Touchscreen, J11 Touchscreen, J12 X-MOTOR, J13 MS1, J14 MS0, J15 Y-MOTOR, J16 MS1, J17 MS0, J2 Z-DRIVE, J3 ISP, J4 UART, J5 12V Supply, J6 MicroSD Card, J7 HWB, J8 USB-6PSMT, J9 Home Switches, Q1 16MHz

Commit message: Start of major restructure using ATmega328
Parts:
- removed C7, C8: 100nF, freetronics-master-v1:CAP0603
- removed C9: 1µF, freetronics-master-v1:CAP0603
- removed D3: CDBA120, freetronics-luke:SCHOTTKY
- removed IC5: ATmega32U4, freetronics-jon:ATMEGA32U4-QFN
- removed J1: SERVO, con-molex:22-23-2031
- removed J12: X-MOTOR, con-phoenix-254:MPT4
- removed J15: Y-MOTOR, con-phoenix-254:MPT4
- removed J2: Z-DRIVE, con-phoenix-254:MPT5
- removed J3: ISP, SparkFun:AVR_SPI_PRG_6NS
- removed J4: UART, pinhead:PINHD-1X4
- removed J6: MicroSD Card, RAMPSdisplay:ADAFRUIT_MICROSD
- removed J7: HWB, freetronics-luke:SJ
- removed J8: USB-6PSMT, freetronics-jon:USB-6PSMT
- removed J9: Home Switches, con-phoenix-254:MPT6
- removed LED4: Z, freetronics-master-v1:LED0603
- removed LED5: Y, freetronics-master-v1:LED0603
- removed LED6: X, freetronics-master-v1:LED0603
- removed LED8: SD, freetronics-master-v1:LED0603
- removed R11, R4, R5, R6: 1k, freetronics-master-v1:RESISTOR0603
- removed R17, R18, R19: 10k, freetronics-master-v1:RESISTOR0603
- added C38, C41, C43, C44: 100nF 0603, freetronics:CAP0603
- added C39, C40: 22pF 0603, freetronics:CAP0603
- added C42: 1uF 0603, freetronics:CAP0603
- added CD1: M01PTH, freetronics-2:M01PTH
- added IC10: LM358D, linear:LM358D
- added IC9: ATMEGA16U2-MU, freetronics-jon:ATMEL_ATMEGA8U2-MUQFN
- added JP1, JP2: (no value), freetronics-master-v1:M04SCREW
- added JP3: (no value), freetronics-master-v1:M04PTH
- added L3: 0805 INDUCTOR, freetronics-master-v1:INDUCTOR0805-LARGE
- added LED11: TX/YEL, freetronics:LED0603
- added LED9: RX/GRN, freetronics:LED0603
- added P1: microSD, freetronics-master-v1:USD-SOCKETNEW
- added P2: ICSP:MAIN, pinhead:PINHD-2X3
- added P3: ICSP:USB, pinhead:PINHD-2X3
- added P5: USB-6PSMT, freetronics-jon:USB-6PSMT
- added R48: 27R 0603, freetronics:RESISTOR0603
- added RN1: 2K2, freetronics-master-v1:4R-NCAY16
- added RN2, RN3: 1K, freetronics-master-v1:4R-NCAY16
- added RN4: 10K, freetronics-master-v1:4R-NCAY16
- added S7: RESET, freetronics-master-v1:TAC_SWITCH_2PIN
- added SJ1: GROUND, freetronics-jon:SJCN
- added SJ2: UBOOT, jumper:SJ
- added SJ3: RESET-EN, freetronics-jon:SJCN
- added X1, X3: 16MHz, freetronics-master-v1:CRYSTALHC49UV
- added Z2: PGB1010603, freetronics:RESISTOR0603
- C10: value 100nF -> 22pF 0603; device freetronics-master-v1:CAP0603 -> freetronics:CAP0603
- C11: value 22pF -> 22pF 0603; device freetronics-master-v1:CAP0603 -> freetronics:CAP0603
- C12: value 22pF -> 100nF 0603; device freetronics-master-v1:CAP0603 -> freetronics:CAP0603
- F1: value 500mA -> 500mA PTC 1812; device freetronics-luke:PTC -> rcl:L-EUL1812
- IC1: value HEF4050B -> ATMEGA328P TQFP32; device 40xx:4050D -> freetronics-2:AVR-MEGA8-AI
- IC3: value LD111733 -> LD111733 SOT-223
- Q1: value 16MHz -> FDN340P; device freetronics-master-v1:CRYSTALHC49US -> freetronics-master-v1:MOSFET-PCHANNEL
- R13: value 10k -> 1M 0603; device freetronics-master-v1:RESISTOR0603 -> freetronics:RESISTOR0603
- R14: value 10k -> 22R 0603; device freetronics-master-v1:RESISTOR0603 -> freetronics:RESISTOR0603
- R15: value 22R -> 22R 0603; device freetronics-master-v1:RESISTOR0603 -> freetronics:RESISTOR0603
- R16: value 22R -> 1M 0603; device freetronics-master-v1:RESISTOR0603 -> freetronics:RESISTOR0603
- Z1: value PGB102ST23 -> PGB1010603; device freetronics-luke:PGB102ST23 -> freetronics:RESISTOR0603
Connections:
- removed net !RESET: IC5./RESET, J3.5, R14.1
- removed net !SD_CS: IC1C.I, IC5.PD7(OC4D/ADC10/T0), R13.1
- removed net +5V: C24.1, C36.1, C4.1, C5.1, C8.2, D1.K, D3.K, IC3.VIN, IC4A.OE, IC4P.VDD, IC5.AVCC, IC5.AVCC1, IC5.UVCC, IC5.VCC, IC5.VCC1, IC6.VCC, IC7.VCC, J1-2.S, J2-3.1, J3.2, J4.1, J9-1.1, J9-3.1, J9-5.1, LCD1.VDD, R1.2, R12.2, R13.2, R14.2, R2.2, R20.2, R21.2, R22.2, R23.2, R24.2, R25.2, R3.2, R34.2, R35.2, R36.2, R37.2, R38.2, R39.2, VR1.A
- removed net FOO: IC1C.O, J6.CS, LED8.C
- removed net HWB: IC5.PE2(HWB), J7.2
- removed net LCD_CLOCK: IC4A.CLK, IC5.PD4(ICP1/ADC8)
- removed net LCD_DATA: IC4A.D, IC5.PD0(INT0/OC0B/SCL)
- removed net LCD_STROBE: IC4A.STR, IC5.PD1(INT1/SDA)
- removed net MISO: IC5.PB3(PDO/MISO), J3.1, J6.DATA_OUT
- removed net MOSI: IC1A.I, IC5.PB2(PDI/MOSI), J3.4
- removed net MOSI_3.3V: IC1A.O, J6.DATA_IN
- removed net N$12: LED4.A, R4.1
- removed net N$2: F1.P$1, J8.VBUS
- removed net N$33: J8.D+, R16.2, Z1.P$1
- removed net N$34: J8.D-, R15.2, Z1.P$2
- removed net N$35: C11.2, IC5.XTAL1, Q1.2
- removed net N$39: LED5.A, R5.1
- removed net N$41: LED6.A, R6.1
- removed net N$5: IC7.BOUT1, J15-3.1
- removed net RXD: IC5.PD2(INT2/RXD1), J4.3
- removed net SCK: IC1B.I, IC1D.I, IC5.PB1(SCK), J3.3
- removed net SCK_3.3V: IC1B.O, J6.SCLK
- removed net SERVO: IC5.PD6(T1/OC4D/ADC9), J1-3.S
- removed net TOUCH1: IC5.PF7(ADC7(TDI), J10.1, J11.Y1
- removed net TOUCH2: IC5.PF6(ADC6/TDO), J10.2, J11.X2
- removed net TOUCH3: IC5.PF5(ADC5/TMS), J10.3, J11.Y2
- removed net TOUCH4: IC5.PF4(ADC4/TCK), J10.4, J11.X1
- removed net TXD: IC5.PD3(INT3/TXD1), J4.4
- removed net VDD: C6.1, IC1P.VDD, IC3.VOUT, J6.VDD
- removed net X_DIR: IC5.PB7(OC0A/OC1C/RTS), IC6.DIR
- removed net X_HOME: IC5.PF0(ADC0), J9-2.1, R17.1, R6.2
- removed net X_STEP: IC5.PB6(OC1B/!OC4B!/ADC13), IC6.STEP
- removed net Y_DIR: IC5.PB5(OC1A/!OC4B!/ADC12), IC7.DIR
- removed net Y_HOME: IC5.PF1(ADC1), J9-4.1, R18.1, R5.2
- removed net Y_STEP: IC5.PB4(ADC11), IC7.STEP
- removed net Z_DIR: IC5.PC6(OC3A/!OC4A!), J2-4.1
- removed net Z_HOME: IC5.PE6, J9-6.1, R19.1, R4.2
- removed net Z_STEP: IC5.PC7(ICP3/CLK0/OC4A), J2-5.1
- new net +3V3: C6.1, IC3.VOUT
- new net 3V3D: C44.1, IC10A.-IN, P1.VCC
- new net 5V: C12.1, C24.1, C36.1, C4.1, C41.1, C43.1, C5.1, D1.K, IC1.AVCC, IC1.VCC@1, IC1.VCC@2, IC10P.V+, IC3.VIN, IC4A.OE, IC4P.VDD, IC6.VCC, IC7.VCC, IC9.AVCC, IC9.VCC, JP3.1, LCD1.VDD, LED11.A, LED9.A, P2.2, P3.2, Q1.S, R1.2, R12.2, R2.2, R20.2, R21.2, R22.2, R23.2, R24.2, R25.2, R3.2, R34.2, R35.2, R36.2, R37.2, R38.2, R39.2, RN4A.2, RN4B.2, VR1.A
- new net A0: IC1.PC0(ADC0), J10.1, J11.Y1
- new net A1: IC1.PC1(ADC1), J10.2, J11.X2
- new net A2: IC1.PC2(ADC2), J10.3, J11.Y2
- new net A3: IC1.PC3(ADC3), J10.4, J11.X1
- new net A4_SDA: IC1.PC4(ADC4/SDA)
- new net A5_SCL: IC1.PC5(ADC5/SCL)
- new net A6: IC1.ADC6
- new net A7: IC1.ADC7
- new net AREF: IC1.AREF
- new net D0_RX: IC1.PD0(RXD), JP3.2, RN3D.1
- new net D10_SS: IC1.PB2(SS/OC1B)
- new net D11_MOSI: IC1.PB3(MOSI/OC2), P2.4, RN2C.2
- new net D12_MISO: IC1.PB4(MISO), P1.DO, P2.1
- new net D13_SCK: IC1.PB5(SCK), P2.3, RN2B.2
- new net D1_TX: IC1.PD1(TXD), JP3.3, RN3C.1
- new net D2: IC1.PD2(INT0), IC4A.STR
- new net D3: IC1.PD3(INT1), IC4A.D
- new net D4: IC1.PD4(XCK/T0), IC4A.CLK
- new net D5: IC1.PD5(T1), IC6.DIR
- new net D6: IC1.PD6(AIN0), IC6.STEP
- new net D7: IC1.PD7(AIN1), IC7.DIR
- new net D8: IC1.PB0(ICP), IC7.STEP
- new net D9: IC1.PB1(OC1A), RN2D.2
- new net DTR: IC9.(CTS)PD7, SJ2.2, SJ3.1
- new net MISO2: IC9.(MISO)PB3, P3.1
- new net MOSI2: IC9.(MOSI)PB2, P3.4
- new net N$113: C39.2, IC9.XTAL2, R16.2, X1.2
- new net N$114: C40.2, R16.1, R48.2, X1.1
- new net N$115: F1.1, P5.VBUS
- new net N$117: C42.1, IC9.UCAP
- new net N$77: IC7.AOUT1, JP2.4
- new net N$81: IC10A.OUT, IC10B.+IN
- new net N$82: P1.CS, RN1A.2, RN2D.1
- new net N$83: P1.DI, RN1C.2, RN2C.1
- new net N$84: P1.SCK, RN1B.2, RN2B.1
- new net N$87: CD1.1, P1.CD1
- new net N$88: LED11.C, RN3A.1
- new net N$89: LED9.C, RN3B.1
- new net N$90: C38.1, SJ3.2
- new net RD+: IC9.D+, R15.1
- new net RD-: IC9.D-, R14.1
- new net RESET: C38.2, IC1.PC6(/RESET), P2.5, RN4B.1, S7.S
- new net RESET2: IC9.RESET, P3.5, RN4A.1
- new net SCK2: IC9.(SCLK)PB1, P3.3
- new net USBGND: IC9.UGND, L3.2, P5.GND, SJ1.1
- new net USBRXD: IC9.(TXD1)PD3, RN3D.2
- new net USBTXD: IC9.(RXD1)PD2, RN3C.2
- new net USBVCC: F1.2, IC9.UVCC, Q1.D
- net +12V: now also RN4C.1; no longer J2-1.1
- net GND: now also C12.2, C39.1, C40.1, C41.2, C42.2, C43.2, C44.2, IC1.AGND, IC1.GND@1, IC1.GND@2, IC10P.V-, IC9.GND, IC9.PAD, JP3.4, P1.CD2, P1.GND, P1.SHIELD1, P1.SHIELD2, P2.6, P3.6, RN1A.1, RN1B.1, RN1C.1, RN4D.1, S7.P, SJ1.2, SJ2.1; no longer C12.1, C7.2, C8.1, C9.1, IC1E.I, IC1F.I, IC1P.VSS, IC5.GND, IC5.GND1, IC5.GND2, IC5.GND3, IC5.TGND, IC5.UGND, J1-1.S, J2-2.1, J3.6, J4.2, J6.GND, J6.GND1, J6.VSS, J7.1, J8.FIX1, J8.FIX2, J8.GND, J8.PIN1, J8.PIN2, J8.TAB1, J8.TAB2, LED4.C, LED5.C, LED6.C, R17.2, R18.2, R19.2, Z1.P$3
- net N$1: now also IC7.BOUT1, JP2.2; no longer IC7.AOUT1, J15-1.1
- net N$11: now also IC1.PB6(XTAL1/TOSC1), R13.2, X3.2; no longer IC5.AREF
- net N$21: now also JP1.1; no longer J12-4.1
- net N$22: now also JP1.2; no longer J12-3.1
- net N$23: now also JP1.3; no longer J12-2.1
- net N$28: now also C11.2, IC1.PB7(XTAL2/TOSC2), R13.1, X3.1; no longer C9.2, IC5.UCAP
- net N$3: now also JP1.4; no longer J12-1.1
- net N$36: now also IC9.XTAL1, R48.1; no longer C12.2, IC5.XTAL2, Q1.1
- net N$37: now also L3.1, P5.FIX1, P5.FIX2, P5.PIN1, P5.PIN2, P5.TAB1, P5.TAB2, Z1.2, Z2.2; no longer IC5.D+, R16.1
- net N$38: now also P5.D+, R15.2, Z1.1; no longer IC5.D-, R15.1
- net N$4: now also JP2.1; no longer J15-4.1
- net N$40: now also P5.D-, R14.2, Z2.1; no longer C7.1, D3.A, F1.P$2, IC5.VBUS
- net N$6: now also JP2.3; no longer J15-2.1
- net N$62: now also IC10A.+IN, RN4C.2, RN4D.2; no longer LED8.A, R11.1
- net N$63: now also IC10B.-IN, IC10B.OUT, Q1.G; no longer IC1D.O, R11.2
- net RXLED: now also IC9.PD4, RN3B.2; no longer IC5.PB0(SS)
- net TXLED: now also IC9.(XCK)PD5, RN3A.2; no longer IC5.PD5(XCK/CTS)
Other:
- note added: "!SD_CS"
- note added: "(C) 2013 Freetronics Pty Ltd"
- note added: "(Linked)"
- note added: "ATmega16U2 Microcontroller"
- note added: "ATmega328P Microcontroller"
- note added: "BUTTONS"
- note added: "D"
- note added: "DCInput/USBVCC Auto-switch"
- note added: "G"
- note added: "In Circuit Serial Programming"
- note added: "LCD_CLK"
- note added: "LCD_DATA"
- note added: "LCD_STROBE"
- note added: "RXD"
- note added: "S"
- note added: "SERVO"
- note added: "Stepper 1"
- note added: "Stepper 2"
- note added: "TOUCH1"
- note added: "TOUCH2"
- note added: "TOUCH3"
- note added: "TOUCH4"
- note added: "TXD"
- note added: "X_DIR"
- note added: "X_HOME"
- note added: "X_STEP"
- note added: "Y_DIR"
- note added: "Y_HOME"
- note added: "Y_STEP"
- note added: "Z_HOME"
- note added: "micro SD Card Slot"
- note added: "uSD_nCS"
- note removed: "(C) 2012 Luke Weston"
- note removed: "1812"
- note removed: "44-TQFP"
- note removed: "568-1688-5-ND"
- note removed: "A0"
- note removed: "A1"
- note removed: "A2"
- note removed: "A3"
- note removed: "A4"
- note removed: "A5"
- note removed: "Amphenol 101-00660-68-6"
- note removed: "D0"
- note removed: "D1"
- note removed: "D10"
- note removed: "D11"
- note removed: "D12"
- note removed: "D13"
- note removed: "D2"
- note removed: "D3"
- note removed: "D4"
- note removed: "D5"
- note removed: "D6"
- note removed: "D7"
- note removed: "D8"
- note removed: "D9"
- note removed: "Digi-Key 101-00660-68-6-1-ND"
- note removed: "F2596CT-ND"
- note removed: "HC49US"
- note removed: "IC3: 497-1241-1-ND"
- note removed: "Micro-SD card socket"
- note removed: "Red"
- note removed: "SOT-223"
- note removed: "SOT-23"
- note removed: "Z1:"
- moved on the sheet: C1, C10, C11, C12, C13, C14, C15, C16, C17, C18, C19, C2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

Commit message: Routing for v1.0 release
Parts:
- removed C13, C25: 100uF, rcl:CPOL-EUE2.5-6
- removed IC9: ATMEGA16U2-MU, freetronics-jon:ATMEL_ATMEGA8U2-MUQFN
- removed J10: Touchscreen, pinhead:PINHD-1X4
- removed J11: Touchscreen, SparkFun:DS_TOUCH_CONNECTOR
- removed LED11: TX/YEL, freetronics:LED0603
- removed LED7: 12, freetronics-master-v1:LED0603
- removed LED9: RX/GRN, freetronics:LED0603
- removed RN3: 1K, freetronics-master-v1:4R-NCAY16
- removed RN4: 10K, freetronics-master-v1:4R-NCAY16
- added C7, C8: 100uF 25V, rcl:CPOL-EUD
- added IC5: DRV8811, eje-components:DRV8811
- added J2: Touchscreen, pinhead:PINHD-1X4
- added J3: Touchscreen, SparkFun:DS_TOUCH_CONNECTOR
- added JP4: Servo1, freetronics-master-v1.1:M03PTH
- added JP5: Servo2, freetronics-master-v1.1:M03PTH
- added JP6: I2C, freetronics-master-v1:M04PTH
- added JP7: (no value), freetronics-master-v1.1:M02PTH
- added LED4: GREEN 0603, freetronics-master-v1:LED0603
- added R11, R17, R18, R4, R5, R6: 10K 0603, freetronics:RESISTOR0603
- added R19, R49: 4K7 0603, freetronics:RESISTOR0603
- C1: value 100uF -> 100uF 25V; device rcl:CPOL-EUE2.5-6 -> rcl:CPOL-EUD
- C14, C16: value 220nF -> 220nF 0603
- C15, C5: value 100nF -> 100nF 0603
- C2: value 47µF -> 47uF 10V 1210
- C3: value 100pF -> 100pF 0603
- C6: value 10µF -> 10uF 10V 0805
- IC7: value DRV8811 -> ATMEGA16U2-MU; device eje-components:DRV8811 -> freetronics-jon:ATMEL_ATMEGA8U2-MUQFN
- JP3: value (none) -> SERIAL
- LED1: value TX -> GREEN/TX 0603
- LED2: value RX -> YELLOW/RX 0603
- LED3: value 5V -> BLUE/5V 0603
- R1, R2: value 1k -> 1K 0603
- R10: value 3k0 -> 3k0 0603
- R3: value 1k -> 1K8 0603
- R32, R33, R46, R47: value 0.20Ω 1W -> 0.2R 1W
- R7: value 4k7 -> 3K9 0603
- R8: value 0.2Ω -> 0.2R 0.5W 1210
- R9: value 1k -> 1k 0603
- VR1, VR2, VR3: value 10kΩ -> 10K
- renumbered IC10 to IC8, J13 to SJ4, J14 to SJ5, J16 to SJ6, J17 to SJ7, J5 to J1, L3 to L2, P5 to P4, S7 to SW1, X1 to XTL1, X3 to XTL2
Connections:
- removed net 3V3D: C44.1, IC8A.-IN, P1.VCC
- removed net N$88: LED11.C, RN3A.1
- removed net N$89: LED9.C, RN3B.1
- net +12V: now also C7.+, C8.+, IC5.VMA, IC5.VMB, R6.2; no longer C13.+, C25.+, IC7.VMA, IC7.VMB, RN4C.1
- net +3V3: now also C44.1, IC8A.-IN, P1.VCC
- net 5V: now also IC5.VCC, IC7.AVCC, JP4.2, JP5.2, JP6.1, R19.2, R4.2, R49.2, R5.2; no longer IC9.AVCC, IC9.VCC, LED11.A, LED9.A, RN4A.2, RN4B.2
- net A0: now also J2.1, J3.Y1; no longer J10.1, J11.Y1
- net A1: now also J2.2, J3.X2; no longer J10.2, J11.X2
- net A2: now also J2.3, J3.Y2; no longer J10.3, J11.Y2
- net A3: now also J2.4, J3.X1; no longer J10.4, J11.X1
- net A4_SDA: now also JP6.2, R19.1
- net A5_SCL: now also JP6.3, R49.1
- net A6: now also JP7.1
- net A7: now also JP7.2
- net D0_RX: now also R18.1; no longer RN3D.1
- net D10_SS: now also JP4.1
- net D11_MOSI: now also JP5.1
- net D1_TX: now also R17.1; no longer RN3C.1
- net D2: now also IC5.DIR; no longer IC4A.STR
- net D3: now also IC6.DIR; no longer IC4A.D
- net D4: now also IC4A.STR; no longer IC4A.CLK
- net D5: now also IC5.STEP; no longer IC6.DIR
- net D7: now also IC4A.D; no longer IC7.DIR
- net D8: now also IC4A.CLK; no longer IC7.STEP
- net DTR: now also IC7.(CTS)PD7; no longer IC9.(CTS)PD7
- net GND: now also C7.-, C8.-, IC5.GND, IC5.GND1, IC5.GND2, IC7.PAD, JP4.3, JP5.3, JP6.4, LED4.C, R11.1; no longer C13.-, C25.-, IC7.GND1, IC7.GND2, IC9.GND, IC9.PAD, LED7.C, RN4D.1
- net MISO2: now also IC7.(MISO)PB3; no longer IC9.(MISO)PB3
- net MOSI2: now also IC7.(MOSI)PB2; no longer IC9.(MOSI)PB2
- net N$1: now also IC6.BOUT1; no longer IC7.BOUT1
- net N$10: now also IC6.VGD; no longer IC7.VGD
- net N$113: now also IC7.XTAL2; no longer IC9.XTAL2
- net N$117: now also IC7.UCAP; no longer IC9.UCAP
- net N$13: now also IC6.ISENA; no longer IC7.ISENA
- net N$14: now also IC6.ISENB; no longer IC7.ISENB
- net N$15: now also IC6.DECAY; no longer IC7.DECAY
- net N$16: now also IC6.RCA; no longer IC7.RCA
- net N$17: now also IC5.CP2; no longer IC6.CP2
- net N$18: now also IC5.CP1; no longer IC6.CP1
- net N$19: now also IC5.SR; no longer IC6.SR
- net N$20: now also IC6.RCB; no longer IC7.RCB
- net N$21: now also IC5.BOUT2; no longer IC6.BOUT2
- net N$22: now also IC5.BOUT1; no longer IC6.BOUT1
- net N$23: now also IC5.AOUT2; no longer IC6.AOUT2
- net N$24: now also IC5.VCP; no longer IC6.VCP
- net N$25: now also IC5.DECAY; no longer IC6.DECAY
- net N$26: now also IC5.VGD; no longer IC6.VGD
- net N$27: now also IC5.RCA; no longer IC6.RCA
- net N$3: now also IC5.AOUT1; no longer IC6.AOUT1
- net N$36: now also IC7.XTAL1; no longer IC9.XTAL1
- net N$4: now also IC6.BOUT2; no longer IC7.BOUT2
- net N$42: now also LED4.A; no longer LED7.A
- net N$46: now also IC5.ISENA; no longer IC6.ISENA
- net N$47: now also IC5.ISENB; no longer IC6.ISENB
- net N$48: now also IC5.RCB; no longer IC6.RCB
- net N$49: now also IC5.SLEEP; no longer IC6.SLEEP
- net N$57: now also IC5.RESET; no longer IC6.RESET
- net N$6: now also IC6.AOUT2; no longer IC7.AOUT2
- net N$62: now also R11.2, R6.1; no longer RN4C.2, RN4D.2
- net N$64: now also IC5.VREF; no longer IC6.VREF
- net N$65: now also IC5.ENABLE; no longer IC6.ENABLE
- net N$66: now also IC5.USM1; no longer IC6.USM1
- net N$67: now also IC5.USM0; no longer IC6.USM0
- net N$68: now also IC6.SLEEP; no longer IC7.SLEEP
- net N$69: now also IC6.RESET; no longer IC7.RESET
- net N$7: now also IC6.CP2; no longer IC7.CP2
- net N$72: now also IC6.VREF; no longer IC7.VREF
- net N$73: now also IC6.ENABLE; no longer IC7.ENABLE
- net N$74: now also IC6.USM1; no longer IC7.USM1
- net N$75: now also IC6.USM0; no longer IC7.USM0
- net N$76: now also IC6.SR; no longer IC7.SR
- net N$77: now also IC6.AOUT1; no longer IC7.AOUT1
- net N$8: now also IC6.CP1; no longer IC7.CP1
- net N$82: now also RN1C.2; no longer RN1A.2
- net N$83: now also RN1B.2; no longer RN1C.2
- net N$84: now also RN1A.2; no longer RN1B.2
- net N$9: now also IC6.VCP; no longer IC7.VCP
- net RD+: now also IC7.D+; no longer IC9.D+
- net RD-: now also IC7.D-; no longer IC9.D-
- net RESET: now also R5.1; no longer RN4B.1
- net RESET2: now also IC7.RESET, R4.1; no longer IC9.RESET, RN4A.1
- net RXLED: now also IC7.PD4; no longer IC9.PD4, RN3B.2
- net SCK2: now also IC7.(SCLK)PB1; no longer IC9.(SCLK)PB1
- net TXLED: now also IC7.(XCK)PD5; no longer IC9.(XCK)PD5, RN3A.2
- net USBGND: now also IC7.UGND; no longer IC9.UGND
- net USBRXD: now also IC7.(TXD1)PD3, R18.2; no longer IC9.(TXD1)PD3, RN3D.2
- net USBTXD: now also IC7.(RXD1)PD2, R17.2; no longer IC9.(RXD1)PD2, RN3C.2
- net USBVCC: now also IC7.UVCC; no longer IC9.UVCC
Other:
- note added: "Change to DRV8825?"
- note added: "Released under the TAPR Open Hardware License: tapr.org/ohl"
- note added: "S1_DIR"
- note added: "S1_STEP"
- note added: "S2_DIR"
- note added: "S2_STEP"
- note added: "StepDuino Stepper Motor Controller"
- note added: "V1.0 (2013-06-29)"
- note added: "www.freetronics.com/stepduino"
- note added: "~"
- note removed: "0.5 W"
- note removed: "0805"
- note removed: "10 V"
- note removed: "10V"
- note removed: "1210"
- note removed: "35V"
- note removed: "73L5R20JCT-ND"
- note removed: "BUTTONS"
- note removed: "Blue"
- note removed: "C2: 445-1409-1-ND"
- note removed: "CNC Plotter Controller"
- note removed: "CP-037A-ND"
- note removed: "Green"
- note removed: "Released under the CERN Open Hardware License: www.ohwr.org/cernohl"
- note removed: "SERVO"
- note removed: "V0.5 (02/06/2012)"
- note removed: "X_DIR"
- note removed: "X_HOME"
- note removed: "X_STEP"
- note removed: "Y_DIR"
- note removed: "Y_HOME"
- note removed: "Y_STEP"
- note removed: "Yellow"
- note removed: "Z_HOME"
- note removed: "github.com/lukeweston/CNCPlotter"
- moved on the sheet: C1, C4, C44, C5, C6, CD1, IC3, IC4, IC4P, IC6, JP3, LCD1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

Commit message: Added documentation and preview image
Parts:
- removed C43, C44: 100nF 0603, freetronics:CAP0603
- removed J3: Touchscreen, SparkFun:DS_TOUCH_CONNECTOR
- added C25: 220nF, freetronics-master-v1:CAP0603
- added C37: 22pF 0603, freetronics:CAP0603
- added C9: 100nF 0603, freetronics:CAP0603
- C1, C8: value 100uF 25V -> 100uF 50V; device rcl:CPOL-EUD -> freetronics-original:CAP_POLE
- C26, C33: value 220nF -> 100nF
- C27, C32: value 100nF -> 220nF
- C28: value 220nF -> 1nF
- C30: value 1nF -> 100nF
- C36: value 100nF -> 100nF 0603; device freetronics-master-v1:CAP0603 -> freetronics:CAP0603
- C38: value 100nF 0603 -> 22pF 0603
- C39: value 22pF 0603 -> 100nF 0603
- C40: value 22pF 0603 -> 1uF 0603
- C42: value 1uF 0603 -> 100nF 0603
- C7: device rcl:CPOL-EUD -> freetronics-original:CAP_POLE
Connections:
- net +12V: now also C25.1; no longer C27.1
- net +3V3: now also C42.1; no longer C44.1
- net 5V: now also C35.1, C39.1; no longer C36.1, C43.1
- net A0: no longer J3.Y1
- net A1: no longer J3.X2
- net A2: no longer J3.Y2
- net A3: no longer J3.X1
- net AREF: now also C9.1
- net GND: now also C26.2, C28.2, C37.1, C38.1, C39.2, C40.2, C9.2; no longer C27.2, C36.2, C39.1, C40.1, C43.2, C44.2
- net N$10: now also C32.1; no longer C33.1
- net N$113: now also C37.2; no longer C39.2
- net N$114: now also C38.2; no longer C40.2
- net N$117: now also C40.1; no longer C42.1
- net N$13: now also C34.1; no longer C35.1
- net N$14: now also C33.1; no longer C34.1
- net N$15: now also C31.1; no longer C32.1
- net N$16: now also C28.1; no longer C29.1
- net N$20: now also C29.1; no longer C30.1
- net N$7: now also C27.2; no longer C28.2
- net N$72: now also C30.1; no longer C31.1
- net N$8: now also C27.1; no longer C28.1
- net N$9: now also C25.2; no longer C26.2
- net N$90: now also C36.1; no longer C38.1
- net RESET: now also C36.2; no longer C38.2
Other:
- note added: "20x4 LCD"
- note added: "3.3V Power Supply"
- note added: "SKU: STEPD"
- note added: "Serial / I2C / Analog Breakouts"
- note added: "Servo Outputs"
- note added: "Status LEDs"
- note added: "V1.1 (2013-09-17)"
- note removed: "V1.0 (2013-06-29)"
- moved on the sheet: C12, C26, C27, C28, C29, C30, C31, C32, C33, C34, C35, C36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
