File: STEPDUINO.sch (EAGLE design)
At the start: 140 parts, among them IC1 ATMEGA328P TQFP32, IC2 MC34063, IC3 LD111733 SOT-223, IC4 74HC4094, IC5 DRV8811, IC6 DRV8811, IC7 ATMEGA16U2-MU, IC8 LM358D, J1 12V Supply, J2 Touchscreen, P1 microSD, P2 ICSP:MAIN, P3 ICSP:USB, P4 USB-6PSMT, Q1 FDN340P, SW1 RESET

Commit message: Made 0603 resistor and capacitor footprints consistent
Parts:
- C10, C11, C12, C36, C37, C38, C39, C40, C41, C42, C9: device freetronics:CAP0603 -> freetronics-master-v1.1:CAP0603
- R1, R2, R3, R7: device freetronics-master-v1:RESISTOR0603 -> freetronics-master-v1.1:RESISTOR0603
- R11, R13, R14, R15, R16, R19, R4, R48, R49, R5, R6, Z1, Z2: device freetronics:RESISTOR0603 -> freetronics-master-v1.1:RESISTOR0603
Changed lines of the file:
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@@
 <?xml version="1.0" encoding="utf-8"?>
 <!DOCTYPE eagle SYSTEM "eagle.dtd">
-<eagle version="6.3">
+<eagle version="6.5.0">
 <drawing>
 <settings>
@@
 <part name="P+11" library="supply1" deviceset="+12V" device=""/>
 <part name="LED4" library="freetronics-master-v1" deviceset="LED" device="0603" value="GREEN 0603"/>
-<part name="R7" library="freetronics-master-v1" deviceset="RESISTOR" device="0603" value="3K9 0603"/>
+<part name="R7" library="freetronics-master-v1.1" deviceset="RESISTOR" device="0603" value="3K9 0603"/>
 <part name="R9" library="freetronics-master-v1" deviceset="RESISTOR" device="0603" value="1k 0603"/>
 <part name="R10" library="freetronics-master-v1" deviceset="RESISTOR" device="0603" value="3k0 0603"/>
 <part name="R8" library="rcl" deviceset="R-EU_" device="R1210" value="0.2R 0.5W 1210"/>
 <part name="R12" library="freetronics-master-v1" deviceset="RESISTOR" device="0603" value="22R"/>
-<part name="R3" library="freetronics-master-v1" deviceset="RESISTOR" device="0603" value="1K8 0603"/>
-<part name="R2" library="freetronics-master-v1" deviceset="RESISTOR" device="0603" value="1K 0603"/>
-<part name="R1" library="freetronics-master-v1" deviceset="RESISTOR" device="0603" value="1K 0603"/>
+<part name="R3" library="freetronics-master-v1.1" deviceset="RESISTOR" device="0603" value="1K8 0603"/>
+<part name="R2" library="freetronics-master-v1.1" deviceset="RESISTOR" device="0603" value="1K 0603"/>
+<part name="R1" library="freetronics-master-v1.1" deviceset="RESISTOR" device="0603" value="1K 0603"/>
 <part name="P+3" library="supply1" deviceset="+5V" device=""/>
 <part name="D2" library="freetronics-luke" deviceset="SCHOTTKY" device="" value="CDBA120"/>
@@
 <part name="GND29" library="SparkFun" deviceset="GND" device=""/>
 <part name="XTL2" library="freetronics-master-v1" deviceset="CRYSTAL" device="HC49UV" value="16MHz"/>
-<part name="C10" library="freetronics" deviceset="CAP" device="0603" value="22pF 0603"/>
-<part name="C11" library="freetronics" deviceset="CAP" device="0603" value="22pF 0603"/>
+<part name="C10" library="freetronics-master-v1.1" deviceset="CAP" device="0603" value="22pF 0603"/>
+<part name="C11" library="freetronics-master-v1.1" deviceset="CAP" device="0603" value="22pF 0603"/>
 <part name="GND31" library="SparkFun" deviceset="GND" device=""/>
-<part name="C12" library="freetronics" deviceset="CAP" device="0603" value="100nF 0603"/>
+<part name="C12" library="freetronics-master-v1.1" deviceset="CAP" device="0603" value="100nF 0603"/>
 <part name="GND32" library="SparkFun" deviceset="GND" device=""/>
 <part name="U$4" library="SparkFun" deviceset="5V" device=""/>
 <part name="U$27" library="SparkFun" deviceset="5V" device=""/>
-<part name="C36" library="freetronics" deviceset="CAP" device="0603" value="100nF 0603"/>
+<part name="C36" library="freetronics-master-v1.1" deviceset="CAP" device="0603" value="100nF 0603"/>
 <part name="SJ3" library="freetronics-jon" deviceset="SJC" device="N" value="RESET-EN"/>
 <part name="SJ2" library="jumper" deviceset="SJ" device="" value="UBOOT"/>
 <part name="GND35" library="SparkFun" deviceset="GND" device=""/>
-<part name="R13" library="freetronics" deviceset="RESISTOR" device="0603" value="1M 0603"/>
+<part name="R13" library="freetronics-master-v1.1" deviceset="RESISTOR" device="0603" value="1M 0603"/>
 <part name="GND36" library="SparkFun" deviceset="GND" device=""/>
 <part name="F1" library="rcl" deviceset="L-EU" device="L1812" value="500mA PTC 1812"/>
 <part name="U$58" library="SparkFun" deviceset="5V" device=""/>
 <part name="XTL1" library="freetronics-master-v1" deviceset="CRYSTAL" device="HC49UV" value="16MHz"/>
-<part name="C37" library="freetronics" deviceset="CAP" device="0603" value="22pF 0603"/>
-<part name="C38" library="freetronics" deviceset="CAP" device="0603" value="22pF 0603"/>
+<part name="C37" library="freetronics-master-v1.1" deviceset="CAP" device="0603" value="22pF 0603"/>
+<part name="C38" library="freetronics-master-v1.1" deviceset="CAP" device="0603" value="22pF 0603"/>
 <part name="GND37" library="SparkFun" deviceset="GND" device=""/>
 <part name="U$59" library="SparkFun" deviceset="5V" device=""/>
-<part name="C39" library="freetronics" deviceset="CAP" device="0603" value="100nF 0603"/>
-<part name="R14" library="freetronics" deviceset="RESISTOR" device="0603" value="22R 0603"/>
-<part name="R15" library="freetronics" deviceset="RESISTOR" device="0603" value="22R 0603"/>
+<part name="C39" library="freetronics-master-v1.1" deviceset="CAP" device="0603" value="100nF 0603"/>
+<part name="R14" library="freetronics-master-v1.1" deviceset="RESISTOR" device="0603" value="22R 0603"/>
+<part name="R15" library="freetronics-master-v1.1" deviceset="RESISTOR" device="0603" value="22R 0603"/>
 <part name="SJ1" library="freetronics-jon" deviceset="SJC" device="N" value="GROUND"/>
 <part name="IC7" library="freetronics-jon" deviceset="ATMEL_ATMEGA8U2-MU" device="QFN" value="ATMEGA16U2-MU"/>
-<part name="R16" library="freetronics" deviceset="RESISTOR" device="0603" value="1M 0603"/>
-<part name="R48" library="freetronics" deviceset="RESISTOR" device="0603" value="27R 0603"/>
-<part name="Z1" library="freetronics" deviceset="RESISTOR" device="0603" value="PGB1010603"/>
-<part name="Z2" library="freetronics" deviceset="RESISTOR" device="0603" value="PGB1010603"/>
+<part name="R16" library="freetronics-master-v1.1" deviceset="RESISTOR" device="0603" value="1M 0603"/>
+<part name="R48" library="freetronics-master-v1.1" deviceset="RESISTOR" device="0603" value="27R 0603"/>
+<part name="Z1" library="freetronics-master-v1.1" deviceset="RESISTOR" device="0603" value="PGB1010603"/>
+<part name="Z2" library="freetronics-master-v1.1" deviceset="RESISTOR" device="0603" value="PGB1010603"/>
 <part name="L2" library="freetronics-master-v1" deviceset="INDUCTOR" device="0805-LARGE" value="0805 INDUCTOR"/>
-<part name="C40" library="freetronics" deviceset="CAP" device="0603" value="1uF 0603"/>
+<part name="C40" library="freetronics-master-v1.1" deviceset="CAP" device="0603" value="1uF 0603"/>
 <part name="GND38" library="SparkFun" deviceset="GND" device=""/>
 <part name="GND39" library="SparkFun" deviceset="GND" device=""/>
@@
 <part name="IC8" library="linear" deviceset="LM358" device="D"/>
 <part name="GND40" library="SparkFun" deviceset="GND" device=""/>
-<part name="C41" library="freetronics" deviceset="CAP" device="0603" value="100nF 0603"/>
+<part name="C41" library="freetronics-master-v1.1" deviceset="CAP" device="0603" value="100nF 0603"/>
 <part name="GND49" library="SparkFun" deviceset="GND" device=""/>
 <part name="U$67" library="SparkFun" deviceset="5V" device=""/>
@@
 <part name="GND3" library="SparkFun" deviceset="GND" device=""/>
 <part name="RN2" library="freetronics-master-v1" deviceset="4R-N" device="CAY16" value="1K"/>
-<part name="C42" library="freetronics" deviceset="CAP" device="0603" value="100nF 0603"/>
+<part name="C42" library="freetronics-master-v1.1" deviceset="CAP" device="0603" value="100nF 0603"/>
 <part name="GND4" library="SparkFun" deviceset="GND" device=""/>
 <part name="CD1" library="freetronics-2" deviceset="M01" device="PTH"/>
@@
 <part name="+3V1" library="supply1" deviceset="+3V3" device="" value="+3.3V"/>
 <part name="+3V3" library="supply1" deviceset="+3V3" device="" value="+3.3V"/>
-<part name="R4" library="freetronics" deviceset="RESISTOR" device="0603" value="10K 0603"/>
-<part name="R5" library="freetronics" deviceset="RESISTOR" device="0603" value="10K 0603"/>
-<part name="R6" library="freetronics" deviceset="RESISTOR" device="0603" value="10K 0603"/>
-<part name="R11" library="freetronics" deviceset="RESISTOR" device="0603" value="10K 0603"/>
+<part name="R4" library="freetronics-master-v1.1" deviceset="RESISTOR" device="0603" value="10K 0603"/>
+<part name="R5" library="freetronics-master-v1.1" deviceset="RESISTOR" device="0603" value="10K 0603"/>
+<part name="R6" library="freetronics-master-v1.1" deviceset="RESISTOR" device="0603" value="10K 0603"/>
+<part name="R11" library="freetronics-master-v1.1" deviceset="RESISTOR" device="0603" value="10K 0603"/>
 <part name="R17" library="freetronics" deviceset="RESISTOR" device="0603" value="10K 0603"/>
 <part name="R18" library="freetronics" deviceset="RESISTOR" device="0603" value="10K 0603"/>
@@
 <part name="GND5" library="SparkFun" deviceset="GND" device=""/>
 <part name="P+19" library="supply1" deviceset="+5V" device=""/>
-<part name="R19" library="freetronics" deviceset="RESISTOR" device="0603" value="4K7 0603"/>
-<part name="R49" library="freetronics" deviceset="RESISTOR" device="0603" value="4K7 0603"/>
+<part name="R19" library="freetronics-master-v1.1" deviceset="RESISTOR" device="0603" value="4K7 0603"/>
+<part name="R49" library="freetronics-master-v1.1" deviceset="RESISTOR" device="0603" value="4K7 0603"/>
 <part name="U$42" library="SparkFun" deviceset="5V" device=""/>
 <part name="JP7" library="freetronics-master-v1.1" deviceset="M02" device="PTH"/>
-<part name="C9" library="freetronics" deviceset="CAP" device="0603" value="100nF 0603"/>
+<part name="C9" library="freetronics-master-v1.1" deviceset="CAP" device="0603" value="100nF 0603"/>
 <part name="GND6" library="SparkFun" deviceset="GND" device=""/>
 </parts>
